Commit message: Update robot xacro, lidar placement, house world, launch and rviz config

File: src/vacuum_robot_description/urdf/vacuum_robot_v2.xacro (robot description, xacro)
@@ -1,39 +1,36 @@
 <?xml version="1.0"?>
 <robot name="vacuum_robot" xmlns:xacro="http://www.ros.org/wiki/xacro">
-  <!-- Parámetros básicos -->
-  <xacro:property name="base_length" value="0.30"/>
-  <xacro:property name="base_width"  value="0.28"/>
+  <xacro:property name="base_radius" value="0.16"/>
   <xacro:property name="base_height" value="0.08"/>
   <xacro:property name="wheel_radius" value="0.035"/>
   <xacro:property name="wheel_width"  value="0.02"/>
-  <xacro:property name="wheel_sep"    value="0.22"/>
-  <xacro:property name="caster_radius" value="0.015"/>
-  <!-- Materiales simples -->
+  <xacro:property name="wheel_separation" value="0.22"/>
+  <xacro:property name="wheel_x" value="-0.055"/>
+  <xacro:property name="wheel_z" value="${wheel_radius}"/>
+  <xacro:property name="caster_radius" value="0.018"/>
+  <xacro:property name="turret_length" value="0.03"/>
+  <xacro:property name="turret_radius" value="0.035"/>
   <material name="gray"><color rgba="0.6 0.6 0.6 1"/></material>
   <material name="black"><color rgba="0.1 0.1 0.1 1"/></material>
-  <!-- BASE -->
   <link name="base_link">
     <visual>
-      <origin xyz="0 0 0.04" rpy="0 0 0"/>
-      <geometry>
-        <cylinder radius="0.16" length="0.08"/>
+      <origin xyz="0 0 ${wheel_radius + base_height/2}" rpy="0 0 0"/>
+      <geometry>
+        <cylinder radius="${base_radius}" length="${base_height}"/>
       </geometry>
       <material name="gray"/>
     </visual>
     <collision>
-      <origin xyz="0 0 0.04" rpy="0 0 0"/>
-      <geometry>
-        <cylinder radius="0.16" length="0.08"/>
-      </geometry>
-    </collision>
-    <inertial>
-      <origin xyz="0 0 0.04" rpy="0 0 0"/>
+      <origin xyz="0 0 ${wheel_radius + base_height/2}" rpy="0 0 0"/>
+      <geometry>
+        <cylinder radius="${base_radius}" length="${base_height}"/>
+      </geometry>
+    </collision>
+    <inertial>
       <mass value="5.0"/>
-      <inertia ixx="0.05" ixy="0.0" ixz="0.0"
-               iyy="0.05" iyz="0.0"
-               izz="0.08"/>
-    </inertial>
-  </link>
-  <!-- RUEDA IZQUIERDA -->
+      <origin xyz="0 0 ${wheel_radius + base_height/2}" rpy="0 0 0"/>
+      <inertia ixx="0.08" ixy="0.0" ixz="0.0" iyy="0.08" iyz="0.0" izz="0.08"/>
+    </inertial>
+  </link>
   <link name="left_wheel_link">
     <visual>
@@ -51,8 +48,7 @@
     </collision>
     <inertial>
-      <mass value="0.2"/>
-      <inertia ixx="0.0002" ixy="0" ixz="0"
-               iyy="0.0002" iyz="0"
-               izz="0.0002"/>
+      <mass value="0.3"/>
+      <origin xyz="0 0 0" rpy="0 0 0"/>
+      <inertia ixx="0.0005" ixy="0" ixz="0" iyy="0.0005" iyz="0" izz="0.0005"/>
     </inertial>
   </link>
@@ -60,8 +56,14 @@
     <parent link="base_link"/>
     <child link="left_wheel_link"/>
-    <origin xyz="0 ${wheel_sep/2} ${wheel_radius}" rpy="0 0 0"/>
+    <origin xyz="${wheel_x} ${wheel_separation/2} ${wheel_z}" rpy="0 0 0"/>
     <axis xyz="0 1 0"/>
   </joint>
-  <!-- RUEDA DERECHA -->
+  <gazebo reference="left_wheel_link">
+    <mu1>0.2</mu1>
+    <mu2>0.2</mu2>
+    <kp>1000000.0</kp>
+    <kd>100.0</kd>
+    <material>Gazebo/Black</material>
+  </gazebo>
   <link name="right_wheel_link">
     <visual>
@@ -79,8 +81,7 @@
     </collision>
     <inertial>
-      <mass value="0.2"/>
-      <inertia ixx="0.0002" ixy="0" ixz="0"
-               iyy="0.0002" iyz="0"
-               izz="0.0002"/>
+      <mass value="0.3"/>
+      <origin xyz="0 0 0" rpy="0 0 0"/>
+      <inertia ixx="0.0005" ixy="0" ixz="0" iyy="0.0005" iyz="0" izz="0.0005"/>
     </inertial>
   </link>
@@ -88,8 +89,14 @@
     <parent link="base_link"/>
     <child link="right_wheel_link"/>
-    <origin xyz="0 ${-wheel_sep/2} ${wheel_radius}" rpy="0 0 0"/>
+    <origin xyz="${wheel_x} -${wheel_separation/2} ${wheel_z}" rpy="0 0 0"/>
     <axis xyz="0 1 0"/>
   </joint>
-  <!-- CASTER (rueda loca / esfera simple) -->
+  <gazebo reference="right_wheel_link">
+    <mu1>0.2</mu1>
+    <mu2>0.2</mu2>
+    <kp>1000000.0</kp>
+    <kd>100.0</kd>
+    <material>Gazebo/Black</material>
+  </gazebo>
   <link name="caster_link">
     <visual>
@@ -108,7 +115,6 @@
     <inertial>
       <mass value="0.05"/>
-      <inertia ixx="0.00001" ixy="0" ixz="0"
-               iyy="0.00001" iyz="0"
-               izz="0.00001"/>
+      <origin xyz="0 0 0" rpy="0 0 0"/>
+      <inertia ixx="0.00001" ixy="0" ixz="0" iyy="0.00001" iyz="0" izz="0.00001"/>
     </inertial>
   </link>
@@ -116,27 +122,28 @@
     <parent link="base_link"/>
     <child link="caster_link"/>
-    <!-- caster al frente -->
-    <origin xyz="${base_length/2 - 0.04} 0 ${caster_radius}" rpy="0 0 0"/>
-  </joint>
-    <!-- Torreta LIDAR (visual) -->
+    <origin xyz="${base_radius - 0.03} 0 ${caster_radius}" rpy="0 0 0"/>
+  </joint>
+  <gazebo reference="caster_link">
+    <mu1>0.3</mu1>
+    <mu2>0.3</mu2>
+  </gazebo>
   <link name="lidar_turret_link">
     <visual>
-      <origin xyz="0 0 0.095" rpy="0 0 0"/>
-      <geometry>
-        <cylinder radius="0.035" length="0.03"/>
-      </geometry>
-      <material name="black"/>
-    </visual>
-    <collision>
-      <origin xyz="0 0 0.095" rpy="0 0 0"/>
-      <geometry>
-        <cylinder radius="0.035" length="0.03"/>
+      <origin xyz="0 0 ${turret_length/2}" rpy="0 0 0"/>
+      <geometry>
+        <cylinder radius="${turret_radius}" length="${turret_length}"/>
+      </geometry>
+      <material name="black"/>
+    </visual>
+    <collision>
+      <origin xyz="0 0 ${turret_length/2}" rpy="0 0 0"/>
+      <geometry>
+        <cylinder radius="${turret_radius}" length="${turret_length}"/>
       </geometry>
     </collision>
     <inertial>
       <mass value="0.1"/>
-      <inertia ixx="0.0001" ixy="0" ixz="0"
-               iyy="0.0001" iyz="0"
-               izz="0.0001"/>
+      <origin xyz="0 0 ${turret_length/2}" rpy="0 0 0"/>
+      <inertia ixx="0.0001" ixy="0" ixz="0" iyy="0.0001" iyz="0" izz="0.0001"/>
     </inertial>
   </link>
@@ -144,39 +151,55 @@
     <parent link="base_link"/>
     <child link="lidar_turret_link"/>
-    <origin xyz="0 0 0" rpy="0 0 0"/>
-  </joint>
-  <!-- Frame del LIDAR (donde luego saldrá /scan) -->
+    <origin xyz="0 0 ${wheel_radius + base_height}" rpy="0 0 0"/>
+  </joint>
   <link name="laser_link"/>
   <joint name="laser_joint" type="fixed">
     <parent link="lidar_turret_link"/>
     <child link="laser_link"/>
-    <origin xyz="0 0 0.015" rpy="0 0 0"/>
-  </joint>
-  <!-- LIDAR Gazebo -->
+    <origin xyz="0 0 ${turret_length + 0.005}" rpy="0 0 0"/>
+  </joint>
   <gazebo reference="laser_link">
-  <sensor type="ray" name="lidar_sensor">
-    <pose>0 0 0 0 0 0</pose>
-    <visualize>true</visualize>
-    <update_rate>10</update_rate>
-    <ray>
-      <scan>
-        <horizontal>
-          <samples>720</samples>
-          <resolution>1</resolution>
-          <min_angle>-3.14159</min_angle>
-          <max_angle>3.14159</max_angle>
-        </horizontal>
-      </scan>
-      <range>
-        <min>0.12</min>
-        <max>8.0</max>
-        <resolution>0.01</resolution>
-      </range>
-    </ray>
-    <plugin name="gazebo_ros_laser" filename="libgazebo_ros_laser.so">
-      <topicName>scan</topicName>
-      <frameName>laser_link</frameName>
+    <sensor type="ray" name="lidar_sensor">
+      <pose>0 0 0 0 0 0</pose>
+      <visualize>true</visualize>
+      <update_rate>10</update_rate>
+      <ray>
+        <scan>
+          <horizontal>
+            <samples>720</samples>
+            <resolution>1</resolution>
+            <min_angle>-3.14159</min_angle>
+            <max_angle>3.14159</max_angle>
+          </horizontal>
+        </scan>
+        <range>
+          <min>0.12</min>
+          <max>8.0</max>
+          <resolution>0.01</resolution>
+        </range>
+      </ray>
+      <plugin name="gazebo_ros_laser" filename="libgazebo_ros_laser.so">
+        <topicName>scan</topicName>
+        <frameName>laser_link</frameName>
+      </plugin>
+    </sensor>
+  </gazebo>
+  <gazebo>
+    <plugin name="diff_drive" filename="libgazebo_ros_diff_drive.so">
+      <leftJoint>left_wheel_joint</leftJoint>
+      <rightJoint>right_wheel_joint</rightJoint>
+      <wheelSeparation>${wheel_separation}</wheelSeparation>
+      <wheelDiameter>${2*wheel_radius}</wheelDiameter>
+      <torque>20</torque>
+      <velocityLimit>2.0</velocityLimit>
+      <updateRate>50</updateRate>
+      <commandTopic>cmd_vel</commandTopic>
+      <odometryTopic>odom</odometryTopic>
+      <odometryFrame>odom</odometryFrame>
+      <robotBaseFrame>base_link</robotBaseFrame>
+      <publishWheelTF>false</publishWheelTF>
+      <publishWheelJointState>false</publishWheelJointState>
+      <publishTf>true</publishTf>
     </plugin>
-  </sensor>
-</gazebo>
+  </gazebo>
 </robot>

Commit message: Modelos y ajustes

File: src/vacuum_robot_description/urdf/vacuum_robot_v2.xacro (robot description, xacro)
@@ -15,9 +15,8 @@
   <link name="base_link">
     <visual>
-      <origin xyz="0 0 ${wheel_radius + base_height/2}" rpy="0 0 0"/>
-      <geometry>
-        <cylinder radius="${base_radius}" length="${base_height}"/>
-      </geometry>
-      <material name="gray"/>
+      <origin xyz="0 0 0" rpy="0 0 0"/>
+      <geometry>
+        <mesh filename="package://vacuum_robot_description/meshes/own_vacuum.dae" scale="0.01 0.01 0.01"/>
+      </geometry>
     </visual>
     <collision>
@@ -105,5 +104,4 @@
         <sphere radius="${caster_radius}"/>
       </geometry>
-      <material name="black"/>
     </visual>
     <collision>
@@ -119,4 +117,7 @@
     </inertial>
   </link>
+  <gazebo reference="caster_link">
+  <material>Gazebo/Black</material>
+  </gazebo>
   <joint name="caster_joint" type="fixed">
     <parent link="base_link"/>
@@ -130,9 +131,8 @@
   <link name="lidar_turret_link">
     <visual>
-      <origin xyz="0 0 ${turret_length/2}" rpy="0 0 0"/>
-      <geometry>
-        <cylinder radius="${turret_radius}" length="${turret_length}"/>
-      </geometry>
-      <material name="black"/>
+      <origin xyz="0 0 0" rpy="0 0 0"/>
+      <geometry>
+        <mesh filename="package://vacuum_robot_description/meshes/lidar.dae" scale="0.01 0.01 0.01"/>
+      </geometry>
     </visual>
     <collision>
@@ -157,5 +157,5 @@
     <parent link="lidar_turret_link"/>
     <child link="laser_link"/>
-    <origin xyz="0 0 ${turret_length + 0.005}" rpy="0 0 0"/>
+    <origin xyz="0 0 ${turret_length - 0.005}" rpy="0 0 0"/>
   </joint>
   <gazebo reference="laser_link">
@@ -174,5 +174,5 @@
         </scan>
         <range>
-          <min>0.12</min>
+          <min>0.05</min>
           <max>8.0</max>
           <resolution>0.01</resolution>
